File: PCB/PCB_V2/PCB_V2/MP1584ENCircuit.kicad_sch (KiCad schematic)
At the start: 0 parts

Commit message: Pushing most recent changes - 10/6/2026
1. Finished the schematics of all the individual modules
2. Made the changes to errors and the hierarchal issues for the MP1584
3. Fixed the open connections for the OLIMEX ESP32 and the labeling for the same

TO DO//
1. Check the current warnings while running ERC (single label warnings and the no connect ones)
2. The tracing and component placement needs to be finalised
3. EMI/EMC placement for the modules needs to be kept in mind with a priority
Parts:
- added C25, C26: 10uF, Capacitor_SMD:C_1206_3216Metric_Pad1.33x1.80mm_HandSolder, symbol Device:C
- added C27: 100nF, Capacitor_SMD:C_0603_1608Metric_Pad1.08x0.95mm_HandSolder, symbol Device:C
- added C28: 220pF, Capacitor_SMD:C_0603_1608Metric_Pad1.08x0.95mm_HandSolder, symbol Device:C
- added C29, C30: 22uF, Capacitor_SMD:C_1206_3216Metric_Pad1.33x1.80mm_HandSolder, symbol Device:C
- added D16: (no value), Diode_SMD:D_SMA_Handsoldering, symbol Device:D
- added L4: 6.8uH, Inductor_SMD:L_6.3x6.3_H3, symbol Device:L
- added R50: 100k, Resistor_SMD:R_0603_1608Metric_Pad0.98x0.95mm_HandSolder, symbol Device:R
- added R51: 24.9k, Resistor_SMD:R_0603_1608Metric_Pad0.98x0.95mm_HandSolder, symbol Device:R
- added R52: 200k, Resistor_SMD:R_0603_1608Metric_Pad0.98x0.95mm_HandSolder, symbol Device:R
- added R53: 68.1k, Resistor_SMD:R_0603_1608Metric_Pad0.98x0.95mm_HandSolder, symbol Device:R
- added U8: MP1584EN, CustomSymbols:SOIC-8_L4.9-W3.9-P1.27-LS6.0-BL-EP3.3, symbol customSymbols:MP1584EN
Connections:
- new net: C27.1, D16.1 (K), L4.1, U8.1 (SW)
- new net: C28.2, R53.1
- new net: R52.1, U8.6 (FREQ)
- new net: C28.1, U8.3 (COMP)
- new net: R50.2, R51.1, U8.2 (EN)
- new net: C27.2, U8.8 (BST)
- new net Feedback: U8.4 (FB)
- new net GND: C25.2, C26.2, C29.2, C30.2, D16.2 (A), R51.2, R52.2, R53.2, U8.5 (GND), U8.9 (GND)
- new net VIN: C25.1, C26.1, R50.1, U8.7 (VIN)
- new net VOUT: C29.1, C30.1, L4.2
