File: PCB/PCB_V3/PCB_V3_Final/PCB_V3_Final.kicad_sch (KiCad schematic)
At the start: 82 parts, among them J1 ESP_Left, J10 LHS_Arrow_+ve, J11 ACS2_pins, J12 ACS4_Pins, J13 ACS2_Screw, J14 ACS4_Screw, J15 MCP_VCC_LINE, J16 AMS_IP_Pins, J17 AMS_OP_Pins, J18 BC1_IN+, J19 BC1_IN-, J2 ESP_Right, J20 BC3_IN+, J21 BC3_IN-, J22 BC1_OUT+, J23 BC1_OUT-, J24 BC3_OUT+, J25 BC3_OUT-, J26 BC2_IN+, J27 BC2_IN-, J28 BC5_IN+, J29 BC5_IN-, J3 ACS1_Pins, J30 BC2_OUT+, J31 BC2_OUT-, J32 BC5_OUT+, J33 BC5_OUT-, J34 LHS_Arrow_-ve, J35 RHS_Arrow_-ve, J36 RHS_Arrow_+ve, J37 LAN8720_pins_1, J4 ACS3_Pins, J44 STATIC_LED_1, J45 STATIC_LED_2, J46 I/P_Terminal, J47 Battery_Terminal, J5 ACS3_Screw, J6 ACS1_Screw, J7 LAN8720_pins_2, J8 MCP_B0, J9 MCP_A0, Q1 IRLZ44N, Q10 IRLZ44N, Q2 IRLZ44N, Q3 IRLZ44N, Q4 IRLZ44N, Q5 IRLZ44N, Q6 IRLZ44N, Q7 IRLZ44N, Q8 IRLZ44N, Q9 IRLZ44N

Commit message: Uploading the final iteration of the PCB design files
Parts:
- removed J11: ACS2_pins, Connector_PinHeader_2.54mm:PinHeader_1x03_P2.54mm_Vertical, symbol Connector:Conn_01x03_Pin
- removed J12: ACS4_Pins, Connector_PinSocket_2.54mm:PinSocket_1x03_P2.54mm_Vertical, symbol Connector:Conn_01x03_Pin
- removed J15: MCP_VCC_LINE, Connector_PinSocket_2.54mm:PinSocket_1x10_P2.54mm_Vertical, symbol Connector:Conn_01x10_Pin
- removed J16: AMS_IP_Pins, Connector_PinSocket_2.54mm:PinSocket_1x02_P2.54mm_Vertical, symbol Connector:Conn_01x02_Pin
- removed J17: AMS_OP_Pins, Connector_PinSocket_2.54mm:PinSocket_1x02_P2.54mm_Vertical, symbol Connector:Conn_01x02_Pin
- removed J18: BC1_IN+, Connector_PinSocket_2.54mm:PinSocket_1x01_P2.54mm_Vertical, symbol Connector:Conn_01x01_Pin
- removed J19: BC1_IN-, Connector_PinSocket_2.54mm:PinSocket_1x01_P2.54mm_Vertical, symbol Connector:Conn_01x01_Pin
- removed J20: BC3_IN+, Connector_PinSocket_2.54mm:PinSocket_1x01_P2.54mm_Vertical, symbol Connector:Conn_01x01_Pin
- removed J25: BC3_OUT-, Connector_PinSocket_2.54mm:PinSocket_1x01_P2.54mm_Vertical, symbol Connector:Conn_01x01_Pin
- removed J30: BC2_OUT+, Connector_PinSocket_2.54mm:PinSocket_1x01_P2.54mm_Vertical, symbol Connector:Conn_01x01_Pin
- removed J31: BC2_OUT-, Connector_PinSocket_2.54mm:PinSocket_1x01_P2.54mm_Vertical, symbol Connector:Conn_01x01_Pin
- removed J34: LHS_Arrow_-ve, Connector_PinSocket_2.54mm:PinSocket_1x05_P2.54mm_Vertical, symbol Connector:Conn_01x05_Pin
- removed J35: RHS_Arrow_-ve, Connector_PinSocket_2.54mm:PinSocket_1x05_P2.54mm_Vertical, symbol Connector:Conn_01x05_Pin
- removed J36: RHS_Arrow_+ve, Connector_PinSocket_2.54mm:PinSocket_1x05_P2.54mm_Vertical, symbol Connector:Conn_01x05_Pin
- removed J37: LAN8720_pins_1, Connector_PinSocket_2.54mm:PinSocket_1x07_P2.54mm_Vertical, symbol Connector:Conn_01x07_Pin
- removed J44: STATIC_LED_1, TerminalBlock_Phoenix:TerminalBlock_Phoenix_MKDS-1,5-2-5.08_1x02_P5.08mm_Horizontal, symbol Connector:Screw_Terminal_01x02
- removed J45: STATIC_LED_2, TerminalBlock_Phoenix:TerminalBlock_Phoenix_MKDS-1,5-2-5.08_1x02_P5.08mm_Horizontal, symbol Connector:Screw_Terminal_01x02
- removed J46: I/P_Terminal, TerminalBlock_Phoenix:TerminalBlock_Phoenix_MKDS-1,5-2-5.08_1x02_P5.08mm_Horizontal, symbol Connector:Screw_Terminal_01x02
- removed J47: Battery_Terminal, TerminalBlock_Phoenix:TerminalBlock_Phoenix_MKDS-1,5-2-5.08_1x02_P5.08mm_Horizontal, symbol Connector:Screw_Terminal_01x02
- removed J7: LAN8720_pins_2, Connector_PinSocket_2.54mm:PinSocket_1x07_P2.54mm_Vertical, symbol Connector:Conn_01x07_Pin
- removed J9: MCP_A0, Connector_PinSocket_2.54mm:PinSocket_1x10_P2.54mm_Vertical, symbol Connector:Conn_01x10_Pin
- added C1: C_Polarized, Capacitor_THT:CP_Radial_D10.0mm_P5.00mm, symbol Device:C_Polarized
- added F1: Fuse, Fuse:Fuseholder_BF020_21.3mmm, symbol Device:Fuse
- added J11: MCP_B0, Connector_PinSocket_2.54mm:PinSocket_1x10_P2.54mm_Vertical, symbol Connector:Conn_01x10_Pin
- added J12: LHS_Arrow_-ve, Connector_PinSocket_2.54mm:PinSocket_1x05_P2.54mm_Vertical, symbol Connector:Conn_01x05_Pin
- added J15: LAN8720_pins_2, Connector_PinSocket_2.54mm:PinSocket_1x07_P2.54mm_Vertical, symbol Connector:Conn_01x07_Pin
- added J16: LAN8720_pins_1, Connector_PinSocket_2.54mm:PinSocket_1x07_P2.54mm_Vertical, symbol Connector:Conn_01x07_Pin
- added J17: MCP_VCC_LINE, Connector_PinSocket_2.54mm:PinSocket_1x10_P2.54mm_Vertical, symbol Connector:Conn_01x10_Pin
- added J18: RHS_Arrow_+ve, Connector_PinSocket_2.54mm:PinSocket_1x05_P2.54mm_Vertical, symbol Connector:Conn_01x05_Pin
- added J19: RHS_Arrow_-ve, Connector_PinSocket_2.54mm:PinSocket_1x05_P2.54mm_Vertical, symbol Connector:Conn_01x05_Pin
- added J20: AMS_IP_Pins, Connector_PinSocket_2.54mm:PinSocket_1x02_P2.54mm_Vertical, symbol Connector:Conn_01x02_Pin
- added J25: AMS_OP_Pins, Connector_PinSocket_2.54mm:PinSocket_1x02_P2.54mm_Vertical, symbol Connector:Conn_01x02_Pin
- added J30: STATIC_LED_1, TerminalBlock_Phoenix:TerminalBlock_Phoenix_MKDS-1,5-2-5.08_1x02_P5.08mm_Horizontal, symbol Connector:Screw_Terminal_01x02
- added J31: STATIC_LED_2, TerminalBlock_Phoenix:TerminalBlock_Phoenix_MKDS-1,5-2-5.08_1x02_P5.08mm_Horizontal, symbol Connector:Screw_Terminal_01x02
- added J34: BC5_IN+, Connector_PinSocket_2.54mm:PinSocket_1x01_P2.54mm_Vertical, symbol Connector:Conn_01x01_Pin
- added J35: BC5_IN-, Connector_PinSocket_2.54mm:PinSocket_1x01_P2.54mm_Vertical, symbol Connector:Conn_01x01_Pin
- added J36: I/P_Terminal, TerminalBlock_Phoenix:TerminalBlock_Phoenix_MKDS-1,5-2-5.08_1x02_P5.08mm_Horizontal, symbol Connector:Screw_Terminal_01x02
- added J37: Battery_Terminal, TerminalBlock_Phoenix:TerminalBlock_Phoenix_MKDS-1,5-2-5.08_1x02_P5.08mm_Horizontal, symbol Connector:Screw_Terminal_01x02
- added J38: BC2_OUT+, Connector_PinSocket_2.54mm:PinSocket_1x01_P2.54mm_Vertical, symbol Connector:Conn_01x01_Pin
- added J39: BC2_OUT-, Connector_PinSocket_2.54mm:PinSocket_1x01_P2.54mm_Vertical, symbol Connector:Conn_01x01_Pin
- added J40: BC5_OUT+, Connector_PinSocket_2.54mm:PinSocket_1x01_P2.54mm_Vertical, symbol Connector:Conn_01x01_Pin
- added J41: BC5_OUT-, Connector_PinSocket_2.54mm:PinSocket_1x01_P2.54mm_Vertical, symbol Connector:Conn_01x01_Pin
- added J7: ACS2_pins, Connector_PinHeader_2.54mm:PinHeader_1x03_P2.54mm_Vertical, symbol Connector:Conn_01x03_Pin
- added J9: ACS4_Pins, Connector_PinSocket_2.54mm:PinSocket_1x03_P2.54mm_Vertical, symbol Connector:Conn_01x03_Pin
- J21: value BC3_IN- -> BC1_IN+
- J22: value BC1_OUT+ -> BC1_IN-
- J23: value BC1_OUT- -> BC3_IN+
- J24: value BC3_OUT+ -> BC3_IN-
- J26: value BC2_IN+ -> BC1_OUT+
- J27: value BC2_IN- -> BC1_OUT-
- J28: value BC5_IN+ -> BC3_OUT+
- J29: value BC5_IN- -> BC3_OUT-
- J32: value BC5_OUT+ -> BC2_IN+
- J33: value BC5_OUT- -> BC2_IN-
- J8: value MCP_B0 -> MCP_A0
Connections:
- net 12V_LR: now also J26.1 (Pin_1); no longer J22.1 (Pin_1)
- net 12V_STATIC1: now also J38.1 (Pin_1)
- net 12V_STATIC2: now also J28.1 (Pin_1); no longer J24.1 (Pin_1)
- net 14.5: now also F1.1, J36.1 (Pin_1); no longer D1.2 (A)
- net 5V: now also J20.1 (Pin_1), J40.1 (Pin_1), J7.3 (Pin_3), J9.3 (Pin_3); no longer J32.1 (Pin_1)
- net A0: now also J8.3 (Pin_3)
- net A1: now also J8.4 (Pin_4)
- net A2: now also J8.5 (Pin_5)
- net A3: now also J8.6 (Pin_6)
- net A4: now also J8.7 (Pin_7)
- net AMS_OP+: now also J16.7 (Pin_7), J17.1 (Pin_1), J17.7 (Pin_7), J25.1 (Pin_1)
- net B0: now also J11.3 (Pin_3); no longer J8.3 (Pin_3)
- net B1: now also J11.4 (Pin_4); no longer J8.4 (Pin_4)
- net B2: now also J11.5 (Pin_5); no longer J8.5 (Pin_5)
- net B3: now also J11.6 (Pin_6); no longer J8.6 (Pin_6)
- net B4: now also J11.7 (Pin_7); no longer J8.7 (Pin_7)
- net D13: now also J17.3 (Pin_3)
- net D17/TX2: now also J15.4 (Pin_4)
- net D18: now also J15.5 (Pin_5)
- net D19: now also J16.2 (Pin_2)
- net D21: now also J15.2 (Pin_2)
- net D22: now also J15.1 (Pin_1)
- net D23: now also J16.5 (Pin_5)
- net D25: now also J15.3 (Pin_3)
- net D26: now also J16.3 (Pin_3)
- net D27: now also J16.4 (Pin_4)
- net D33: now also J9.2 (Pin_2)
- net D35: now also J7.2 (Pin_2)
- net D4: now also J17.4 (Pin_4)
- net GND: now also J22.1 (Pin_1), J24.1 (Pin_1), C1.1, J16.6 (Pin_6), J17.10 (Pin_10), J17.2 (Pin_2), J17.8 (Pin_8), J17.9 (Pin_9), J20.2 (Pin_2), J25.2 (Pin_2), J30.2 (Pin_2), J31.2 (Pin_2), J35.1 (Pin_1), J36.2 (Pin_2), J37.2 (Pin_2), J39.1 (Pin_1), J41.1 (Pin_1), J7.1 (Pin_1), J9.1 (Pin_1); no longer J21.1 (Pin_1), J23.1 (Pin_1)
- net LHS_LED_1: now also J12.1 (Pin_1)
- net LHS_LED_2: now also J12.2 (Pin_2)
- net LHS_LED_3: now also J12.3 (Pin_3)
- net LHS_LED_4: now also J12.4 (Pin_4)
- net LHS_LED_5: now also J12.5 (Pin_5)
- net MAIN_OP: now also J21.1 (Pin_1), J23.1 (Pin_1), J32.1 (Pin_1), J34.1 (Pin_1), J37.1 (Pin_1); no longer J26.1 (Pin_1), J28.1 (Pin_1)
- net RHS_LED_1: now also J19.1 (Pin_1)
- net RHS_LED_2: now also J19.2 (Pin_2)
- net RHS_LED_3: now also J19.3 (Pin_3)
- net RHS_LED_4: now also J19.4 (Pin_4)
- net RHS_LED_5: now also J19.5 (Pin_5)
- net RHS_LED_IP+: now also J18.1 (Pin_1), J18.2 (Pin_2), J18.3 (Pin_3), J18.4 (Pin_4), J18.5 (Pin_5)
- net STATIC1+: now also J31.1 (Pin_1)
- net STATIC2+: now also J30.1 (Pin_1)
- new net: C1.2, D1.2 (A), F1.2

Commit message: Uploading the final PCB files
1. Finished product
2. Made the remaining connections
3. Added the mounting holes for the PCB
4. Final producct --> has to be reviewed in the meeting
Parts:
- added H1, H2, H3, H4: MountingScrew, MountingHole:MountingHole_3.2mm_M3, symbol Auxiliary_Items:MountingScrew

Commit message: Final PCB Upload
1. Made all the changes
2. final PCB files and the gerber files uploaded
Parts:
- removed D1: 1N5822, Diode_THT:D_DO-201AD_P15.24mm_Horizontal, symbol Diode:1N5822
- added D1: D_Schottky, Package_TO_SOT_THT:TO-220-2_Vertical, symbol Device:D_Schottky
- J28: value BC3_OUT+ -> BC3_IN-
Connections:
- net 12V_STATIC1: now also J32.1 (Pin_1); no longer J38.1 (Pin_1)
- net 12V_STATIC2: now also J23.1 (Pin_1); no longer J28.1 (Pin_1)
- net 14.5: no longer R23.1
- net GND: now also C1.2, J28.1 (Pin_1), J38.1 (Pin_1); no longer C1.1, J29.1 (Pin_1), J39.1 (Pin_1)
- net MAIN_OP: now also J29.1 (Pin_1), J39.1 (Pin_1), D1.1 (K); no longer J23.1 (Pin_1), J32.1 (Pin_1)
- net 14.5_VD: now reaches F1.2
- net 14.5_VD: now also C1.1, R23.1, D1.2 (A); no longer C1.2
Other:
- moved on the sheet: C1
